Commit message: Added arm spawning

File: src/test2_description/urdf/test2.urdf (robot description, URDF)
Before this commit: robot test2, 2 links, 1 joints
Links:
- added link base_link, mass 0.1; collision cylinder length=0.02 radius=0.5; visual cylinder length=0.02 radius=0.5
- added link finger1, mass 0.1; collision box size=0.01 0.01 .05; visual box size=0.01 0.01 .05
- added link finger2, mass 0.1; collision box size=0.01 0.01 .05; visual box size=0.01 0.01 .05
- added link link2, mass 0.1; collision cylinder length=0.30 radius=0.03; visual cylinder length=0.30 radius=0.03
- added link link3, mass 0.1; collision cylinder length=0.30 radius=0.03; visual cylinder length=0.30 radius=0.03
- added link link4, mass 0.1; collision box size=0.03 0.03 0.1; visual box size=0.03 0.03 0.1
- added link link5, mass 0.1; collision box size=0.03 0.03 0.1; visual box size=0.03 0.03 0.1
- added link link6, mass 0.1; collision cylinder length=0.10 radius=0.04; visual cylinder length=0.10 radius=0.04
- link link1: mass 1 -> 0.1; geometry collision cylinder length=0.10 radius=0.10; visual cylinder length=0.10 radius=0.10
Joints:
- added joint f_joint1: type prismatic, parent link6, child finger1, origin xyz=0 -0.025 0.1 rpy=0 0 0, axis 0 1 0, limit lower=0.0 upper=0.020 effort=20 velocity=0.2
- added joint f_joint2: type prismatic, parent link6, child finger2, origin xyz=0 0.025 0.1 rpy=0 0 0, axis 0 1 0, limit lower=-0.020 upper=0 effort=20 velocity=0.2
- added joint joint1: type continuous, parent base_link, child link1, origin xyz=0 0 0.01 rpy=0 0 0, axis 0 0 1
- added joint joint2: type revolute, parent link1, child link2, origin xyz=0 0 0.08 rpy=0 0 0, axis 0 1 0, limit lower=-1.57 upper=1.57 effort=100 velocity=1
- added joint joint3: type revolute, parent link2, child link3, origin xyz=0 0 0.28 rpy=0 0 0, axis 0 1 0, limit lower=-2.57 upper=2.57 effort=100 velocity=1
- added joint joint4: type revolute, parent link3, child link4, origin xyz=0 0 0.28 rpy=0 0 0, axis 0 0 1, limit lower=-3.14 upper=3.14 effort=100 velocity=1
- added joint joint5: type revolute, parent link4, child link5, origin xyz=0 0 0.08 rpy=0 0 0, axis 0 1 0, limit lower=-2.57 upper=2.57 effort=100 velocity=1
- added joint joint6: type revolute, parent link5, child link6, origin xyz=0 0 0.08 rpy=0 0 0, axis 1 0 0, limit lower=-2.57 upper=2.57 effort=100 velocity=1
- joint fixed: child link1 -> base_link
