Commit message: Added main.py and fixed initial position

File: src/test2_description/urdf/test2.urdf.xacro (robot description, xacro)
@@ -207,21 +207,29 @@
     </collision>
   </link>
-  <joint name="finger1_base_joint" type="revolute">
+  <!--joint name="finger1_base_joint" type="revolute">
       <parent link="wrist_3_link"/>
       <child link="finger1"/>
       <origin rpy="1.57 1.57 0" xyz="-0.02 0.1 -0.018"/>
-      <axis xyz="1 0 0"/>
+      <axis xyz="1 0 1"/>
       <limit effort="28.0" lower="-3.14159265" upper="3.14159265" velocity="3.2"/>
       <dynamics damping="0.0" friction="0.0"/>
+  </joint-->
+  <joint name="finger1_base_joint" type="prismatic">
+      <parent link="wrist_3_link"/>
+      <child link="finger1"/>
+      <origin rpy="1.57 1.57 0" xyz="-0.02 0.103 -0.018"/>
+      <axis xyz="1 -1 0"/>
+      <limit effort="28.0" lower="-0.2" upper="0.2" velocity="3.2"/>
+      <dynamics damping="0.0" friction="0.0"/>
   </joint>
   <link name="finger1">
     <visual>
         <geometry>
-            <cylinder length="0.04" radius="0.007" />
-        </geometry>
-    </visual>
-    <collision>
-        <geometry>
-            <cylinder length="0.04" radius="0.007" />
+            <cylinder length="0.04" radius="0.004" />
+        </geometry>
+    </visual>
+    <collision>
+        <geometry>
+            <cylinder length="0.04" radius="0.004" />
         </geometry>
     </collision>
@@ -231,21 +239,24 @@
     </inertial>
   </link>
-  <joint name="finger2_base_joint" type="revolute">
+  <gazebo reference="finger1">
+      <material>Gazebo/DarkGrey</material>
+  </gazebo>
+  <joint name="finger2_base_joint" type="prismatic">
       <parent link="wrist_3_link"/>
       <child link="finger2"/>
-      <origin rpy="1.57 1.57 0" xyz="0.02 0.1 -0.018"/>
-      <axis xyz="1 0 0"/>
-      <limit effort="28.0" lower="-3.14159265" upper="3.14159265" velocity="3.2"/>
-    <dynamics damping="0.0" friction="0.0"/>
+      <origin rpy="1.57 1.57 0" xyz="0.02 0.103 -0.018"/>
+      <axis xyz="1 1 0"/>
+      <limit effort="28.0" lower="-0.2" upper="0.2" velocity="3.2"/>
+      <dynamics damping="0.0" friction="0.0"/>
   </joint>
   <link name="finger2">
     <visual>
         <geometry>
-            <cylinder length="0.04" radius="0.007" />
-        </geometry>
-    </visual>
-    <collision>
-        <geometry>
-            <cylinder length="0.04" radius="0.007" />
+            <cylinder length="0.04" radius="0.004" />
+        </geometry>
+    </visual>
+    <collision>
+        <geometry>
+            <cylinder length="0.04" radius="0.004" />
         </geometry>
     </collision>
@@ -255,21 +266,24 @@
     </inertial>
   </link>
-  <joint name="finger3_base_joint" type="revolute">
+  <gazebo reference="finger2">
+      <material>Gazebo/DarkGrey</material>
+  </gazebo>
+  <joint name="finger3_base_joint" type="prismatic">
       <parent link="wrist_3_link"/>
       <child link="finger3"/>
-      <origin rpy="1.57 1.57 0" xyz="0 0.1 0.025"/>
-      <axis xyz="1 0 0"/>
-      <limit effort="28.0" lower="-3.14159265" upper="3.14159265" velocity="3.2"/>
-    <dynamics damping="0.0" friction="0.0"/>
+      <origin rpy="1.57 1.57 0" xyz="0 0.103 0.025"/>
+      <axis xyz="-1 0 0"/>
+      <limit effort="28.0" lower="-0.2" upper="0.2" velocity="3.2"/>
+      <dynamics damping="0.0" friction="0.0"/>
   </joint>
   <link name="finger3">
     <visual>
         <geometry>
-            <cylinder length="0.04" radius="0.007" />
-        </geometry>
-    </visual>
-    <collision>
-        <geometry>
-            <cylinder length="0.04" radius="0.007" />
+            <cylinder length="0.04" radius="0.004" />
+        </geometry>
+    </visual>
+    <collision>
+        <geometry>
+            <cylinder length="0.04" radius="0.004" />
         </geometry>
     </collision>
@@ -279,4 +293,7 @@
     </inertial>
   </link>
+  <gazebo reference="finger3">
+      <material>Gazebo/DarkGrey</material>
+  </gazebo>
   <transmission name="shoulder_pan_trans">
     <type>transmission_interface/SimpleTransmission</type>
@@ -332,4 +349,34 @@
       <mechanicalReduction>1</mechanicalReduction>
     </actuator>
+  </transmission>
+  <transmission name="trans_f_finger">
+      <type>transmission_interface/SimpleTransmission</type>
+      <joint name="finger1_base_joint">
+          <hardwareInterface>hardware_interface/PositionJointInterface</hardwareInterface>
+      </joint>
+      <actuator name="finger1_motor">
+          <hardwareInterface>hardware_interface/PositionJointInterface</hardwareInterface>
+          <mechanicalReduction>1</mechanicalReduction>
+      </actuator>
+  </transmission>
+  <transmission name="trans_finger2">
+      <type>transmission_interface/SimpleTransmission</type>
+      <joint name="finger2_base_joint">
+          <hardwareInterface>hardware_interface/PositionJointInterface</hardwareInterface>
+      </joint>
+      <actuator name="finger2_motor">
+          <hardwareInterface>hardware_interface/PositionJointInterface</hardwareInterface>
+          <mechanicalReduction>1</mechanicalReduction>
+      </actuator>
+  </transmission>
+  <transmission name="trans_finger3">
+      <type>transmission_interface/SimpleTransmission</type>
+      <joint name="finger3_base_joint">
+          <hardwareInterface>hardware_interface/PositionJointInterface</hardwareInterface>
+      </joint>
+      <actuator name="finger3_motor">
+          <hardwareInterface>hardware_interface/PositionJointInterface</hardwareInterface>
+          <mechanicalReduction>1</mechanicalReduction>
+      </actuator>
   </transmission>
   <!-- define the ur5's position and orientation in the world coordinate system -->

Commit message: Added arm movement

File: src/test2_description/urdf/test2.urdf.xacro (robot description, xacro)
@@ -31,5 +31,5 @@
     <origin rpy="0.0 0.0 0.0" xyz="0.0 0.0 0.089159"/>
     <axis xyz="0 0 1"/>
-    <limit effort="150.0" lower="-3.14159265" upper="3.14159265" velocity="3.15"/>
+    <limit effort="150.0" lower="-3.14159265" upper="3.14159265" velocity="0.5"/>
     <dynamics damping="0.0" friction="0.0"/>
   </joint>
@@ -59,5 +59,5 @@
     <origin rpy="0.0 1.570796325 0.0" xyz="0.0 0.13585 0.0"/>
     <axis xyz="0 1 0"/>
-    <limit effort="150.0" lower="-3.14159265" upper="3.14159265" velocity="3.15"/>
+    <limit effort="150.0" lower="-3.14159265" upper="3.14159265" velocity="0.5"/>
     <dynamics damping="0.0" friction="0.0"/>
   </joint>
@@ -87,5 +87,5 @@
     <origin rpy="0.0 0.0 0.0" xyz="0.0 -0.1197 0.425"/>
     <axis xyz="0 1 0"/>
-    <limit effort="150.0" lower="-3.14159265" upper="3.14159265" velocity="3.15"/>
+    <limit effort="150.0" lower="-3.14159265" upper="3.14159265" velocity="0.5"/>
     <dynamics damping="0.0" friction="0.0"/>
   </joint>
@@ -115,5 +115,5 @@
     <origin rpy="0.0 1.570796325 0.0" xyz="0.0 0.0 0.39225"/>
     <axis xyz="0 1 0"/>
-    <limit effort="28.0" lower="-3.14159265" upper="3.14159265" velocity="3.2"/>
+    <limit effort="28.0" lower="-3.14159265" upper="3.14159265" velocity="1.2"/>
     <dynamics damping="0.0" friction="0.0"/>
   </joint>
@@ -143,5 +143,5 @@
     <origin rpy="0.0 0.0 0.0" xyz="0.0 0.093 0.0"/>
     <axis xyz="0 0 1"/>
-    <limit effort="28.0" lower="-3.14159265" upper="3.14159265" velocity="3.2"/>
+    <limit effort="28.0" lower="-3.14159265" upper="3.14159265" velocity="1.2"/>
     <dynamics damping="0.0" friction="0.0"/>
   </joint>
@@ -171,5 +171,5 @@
     <origin rpy="0.0 0.0 0.0" xyz="0.0 0.0 0.09465"/>
     <axis xyz="0 1 0"/>
-    <limit effort="28.0" lower="-3.14159265" upper="3.14159265" velocity="3.2"/>
+    <limit effort="28.0" lower="-3.14159265" upper="3.14159265" velocity="1.2"/>
     <dynamics damping="0.0" friction="0.0"/>
   </joint>
@@ -212,5 +212,5 @@
       <origin rpy="1.57 1.57 0" xyz="-0.02 0.1 -0.018"/>
       <axis xyz="1 0 1"/>
-      <limit effort="28.0" lower="-3.14159265" upper="3.14159265" velocity="3.2"/>
+      <limit effort="28.0" lower="-3.14159265" upper="3.14159265" velocity="1.2"/>
       <dynamics damping="0.0" friction="0.0"/>
   </joint-->
@@ -220,5 +220,5 @@
       <origin rpy="1.57 1.57 0" xyz="-0.02 0.103 -0.018"/>
       <axis xyz="1 -1 0"/>
-      <limit effort="28.0" lower="-0.2" upper="0.2" velocity="3.2"/>
+      <limit effort="5.0" lower="-0.2" upper="0.2" velocity="0.1"/>
       <dynamics damping="0.0" friction="0.0"/>
   </joint>
@@ -247,5 +247,5 @@
       <origin rpy="1.57 1.57 0" xyz="0.02 0.103 -0.018"/>
       <axis xyz="1 1 0"/>
-      <limit effort="28.0" lower="-0.2" upper="0.2" velocity="3.2"/>
+      <limit effort="5.0" lower="-0.2" upper="0.2" velocity="0.1"/>
       <dynamics damping="0.0" friction="0.0"/>
   </joint>
@@ -274,5 +274,5 @@
       <origin rpy="1.57 1.57 0" xyz="0 0.103 0.025"/>
       <axis xyz="-1 0 0"/>
-      <limit effort="28.0" lower="-0.2" upper="0.2" velocity="3.2"/>
+      <limit effort="5.0" lower="-0.2" upper="0.2" velocity="0.1"/>
       <dynamics damping="0.0" friction="0.0"/>
   </joint>
@@ -296,4 +296,76 @@
       <material>Gazebo/DarkGrey</material>
   </gazebo>
+  <link name="camera_link">
+  <visual>
+    <origin xyz="0 0 0" rpy="0 0 0"/>
+    <geometry>
+      <box size="0.01 0.01 0.01"/>
+    </geometry>
+  </visual>
+  <collision>
+    <origin xyz="0 0 0" rpy="0 0 0"/>
+    <geometry>
+      <box size="0.01 0.01 0.01"/>
+    </geometry>
+  </collision>
+  <inertial>
+    <origin xyz="0 0 0" rpy="0 0 0"/>
+    <mass value="0.035"/>
+    <inertia ixx="0.001"  ixy="0"  ixz="0" iyy="0.001" iyz="0" izz="0.001" />
+  </inertial>
+</link>
+<joint name="camera_joint" type="fixed">
+  <parent link="wrist_3_link"/>
+  <child link="camera_link"/>
+  <origin xyz="0 0.08 0" rpy="0 0 1.57"/>
+</joint>
+<!--link name="camera_depth_frame"/>
+<joint name="camera_depth_joint" type="fixed">
+  <origin xyz="0 0 0" rpy="1.57 0 1.57"/>
+  <parent link="camera_link"/>
+  <child link="camera_depth_frame"/>
+</joint-->
+<gazebo reference="camera_link">
+  <material>Gazebo/Wood</material>
+  <sensor name="depth_camera" type="depth">
+    <update_rate>20</update_rate>
+    <camera>
+      <horizontal_fov>1.047198</horizontal_fov>
+      <image>
+        <width>640</width>
+        <height>480</height>
+        <format>R8G8B8</format>
+      </image>
+      <clip>
+        <near>0.05</near>
+        <far>3</far>
+      </clip>
+    </camera>
+    <plugin name="depth_camera_controller" filename="libgazebo_ros_openni_kinect.so">
+      <baseline>0.2</baseline>
+      <alwaysOn>true</alwaysOn>
+      <updateRate>1.0</updateRate>
+      <cameraName>camera</cameraName>
+      <imageTopicName>/test2/color/image_raw</imageTopicName>
+      <cameraInfoTopicName>/test2/color/camera_info</cameraInfoTopicName>
+      <depthImageTopicName>/test2/depth/image_raw</depthImageTopicName>
+      <depthImageInfoTopicName>/test2/depth/camera_info</depthImageInfoTopicName>
+      <pointCloudTopicName>/test2/depth/points</pointCloudTopicName>
+      <frameName>test2</frameName>
+      <pointCloudCutoff>0.5</pointCloudCutoff>
+      <pointCloudCutoffMax>3.0</pointCloudCutoffMax>
+      <distortionK1>0.00000001</distortionK1>
+      <distortionK2>0.00000001</distortionK2>
+      <distortionK3>0.00000001</distortionK3>
+      <distortionT1>0.00000001</distortionT1>
+      <distortionT2>0.00000001</distortionT2>
+      <CxPrime>0</CxPrime>
+      <Cx>0</Cx>
+      <Cy>0</Cy>
+      <focalLength>0</focalLength>
+      <hackBaseline>0</hackBaseline>
+    </plugin>
+  </sensor>
+</gazebo>
   <transmission name="shoulder_pan_trans">
     <type>transmission_interface/SimpleTransmission</type>
