Commit message: Added Inverse Kinematic

File: src/test2_description/urdf/grasper.urdf (robot description, URDF)
Before this commit: robot smart_grasping_sandbox, 35 links, 34 joints
Joints:
- joint world_joint: origin xyz=0.0 0.0 0.1 rpy=0.0 0.0 0.0 -> xyz=0.0 0.0 0.1 rpy=0.0 3.14 3.14

Commit message: Fix inverse kinematics matrix

File: src/test2_description/urdf/grasper.urdf (robot description, URDF)
Before this commit: robot smart_grasping_sandbox, 35 links, 34 joints
Joints:
- joint world_joint: origin xyz=0.0 0.0 0.1 rpy=0.0 3.14 3.14 -> xyz=0.0 0.0 0.1 rpy=0.0 0.0 0.0

Commit message: added yolo recognition

File: src/test2_description/urdf/grasper.urdf (robot description, URDF)
Before this commit: robot smart_grasping_sandbox, 35 links, 34 joints
Links:
- added link camera_link, mass 1e-5; visual box size=0.015 0.015 0.015
Joints:
- added joint camera_joint: type fixed, parent wrist_3_link, child camera_link, origin xyz=0 0.2 0 rpy=-1.57 0 1.57, axis 0 1 0

Commit message: Final camera fix: color adjustemnt and rotation

File: src/test2_description/urdf/grasper.urdf (robot description, URDF)
Before this commit: robot smart_grasping_sandbox, 36 links, 35 joints
Joints:
- joint camera_joint: origin xyz=0 0.2 0 rpy=-1.57 0 1.57 -> xyz=0 0.2 0 rpy=-3.14 0 1.57

Commit message: Automation implementation, rotation range doubled

File: src/test2_description/urdf/grasper.urdf (robot description, URDF)
Before this commit: robot smart_grasping_sandbox, 36 links, 35 joints
Joints:
- joint shoulder_pan_joint: limit lower=-3.14159265359 upper=3.14159265359 effort=330.0 velocity=2.16 -> lower=-6.28318530718 upper=6.28318530718 effort=330.0 velocity=2.16
- joint wrist_1_joint: limit lower=-3.14159265359 upper=3.14159265359 effort=54.0 velocity=3.2 -> lower=-6.28318530718 upper=6.28318530718 effort=54.0 velocity=3.2
- joint wrist_2_joint: limit lower=-3.14159265359 upper=3.14159265359 effort=54.0 velocity=3.2 -> lower=-6.28318530718 upper=6.28318530718 effort=54.0 velocity=3.2
- joint wrist_3_joint: limit lower=-3.14159265359 upper=3.14159265359 effort=54.0 velocity=3.2 -> lower=-6.28318530718 upper=6.28318530718 effort=54.0 velocity=3.2

Commit message: Added bricks grounds, fixed final movement

File: src/test2_description/urdf/grasper.urdf (robot description, URDF)
Before this commit: robot smart_grasping_sandbox, 36 links, 35 joints
Joints:
- joint shoulder_pan_joint: limit lower=-6.28318530718 upper=6.28318530718 effort=330.0 velocity=2.16 -> lower=-6.28318530718 upper=6.28318530718 effort=330.0 velocity=6

Commit message: Fixed bricks rotations

File: src/test2_description/urdf/grasper.urdf (robot description, URDF)
Before this commit: robot smart_grasping_sandbox, 36 links, 35 joints
Joints:
- joint wrist_3_joint: limit lower=-6.28318530718 upper=6.28318530718 effort=54.0 velocity=3.2 -> lower=-6.28318530718 upper=6.28318530718 effort=54.0 velocity=5.4

Commit message: Initial final version

File: src/test2_description/urdf/grasper.urdf (robot description, URDF)
Before this commit: robot smart_grasping_sandbox, 36 links, 35 joints
Joints:
- joint shoulder_lift_joint: limit lower=-3.14159265359 upper=3.14159265359 effort=330.0 velocity=2.16 -> lower=-3.14159265359 upper=3.14159265359 effort=330.0 velocity=3
- joint shoulder_pan_joint: limit lower=-6.28318530718 upper=6.28318530718 effort=330.0 velocity=6 -> lower=-6.28318530718 upper=6.28318530718 effort=330.0 velocity=4
